File: hardware/schematic-pcb/PQopen Device Rail-Mount.kicad_pcb (KiCad board)
At the start: 2 copper layers, 155 x 86.5 mm, 62 parts, among them J1 Conn_01x04, J2 Conn_01x06, J3 Conn_01x22, J4 External Power in 9-36V, J5 5V Output, U1 MCP6022, U2 MCP6022, U3 MCP6022, U4 MCP6022

Commit message: hardware: minor improvements
Parts:
- added H1: MountingHole, MountingHole:MountingHole_2.7mm_M2.5_ISO14580, F.Cu at (142.0, 118.5)
