File: hardware/schematic-pcb/PQopen Device Rail-Mount.kicad_sch (KiCad schematic)
At the start: 62 parts, among them J1 Conn_01x04, J2 Conn_01x06, J3 Conn_01x22, J4 External Power in 9-36V, J5 5V Output, U1 MCP6022, U2 MCP6022, U3 MCP6022, U4 MCP6022

Commit message: hardware: minor improvements
Parts:
- added H1: MountingHole, MountingHole:MountingHole_2.7mm_M2.5_ISO14580, symbol Mechanical:MountingHole
- R18:  mpn (none) -> KTR18EZPF4703; Article KTR18EZPF4703 -> (none)
Changed lines of the file:
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@@
+	)
+	(symbol
+		(lib_id "Mechanical:MountingHole")
+		(at 158.75 179.07 0)
+		(unit 1)
+		(exclude_from_sim yes)
+		(in_bom no)
+		(on_board yes)
+		(dnp no)
+		(fields_autoplaced yes)
+		(property "Reference" "H1"
+			(at 161.29 177.8578 0)
+			(effects
+				(font
+					(size 1.27 1.27)
+				)
+				(justify left)
+			)
+		)
+		(property "Value" "MountingHole"
+			(at 161.29 180.2821 0)
+			(effects
+				(font
+					(size 1.27 1.27)
+				)
+				(justify left)
+			)
+		)
+		(property "Footprint" "MountingHole:MountingHole_2.7mm_M2.5_ISO14580"
+			(at 158.75 179.07 0)
+			(effects
+				(font
+					(size 1.27 1.27)
+				)
+				(hide yes)
+			)
+		)
+		(property "Datasheet" "~"
+			(at 158.75 179.07 0)
+			(effects
+				(font
+					(size 1.27 1.27)
+				)
+				(hide yes)
+			)
+		)
+		(property "Description" "Mounting Hole without connection"
+			(at 158.75 179.07 0)
+			(effects
+				(font
+					(size 1.27 1.27)
+				)
+				(hide yes)
+			)
+		)
+		(instances
+			(project ""
+				(path "/861966a9-b3d2-4fe6-94f3-e5b8424e658f"
+					(reference "H1")
+					(unit 1)
+				)
+			)
+		)
 	)
 	(symbol
@@
 			)
 		)
-		(property "Article" "KTR18EZPF4703"
+		(property " mpn" "KTR18EZPF4703"
 			(at 67.31 87.63 90)
 			(effects
